File: hardware/cantoto.kicad_pcb (KiCad board)
At the start: 2 copper layers, 57 x 41 mm, 56 parts, among them J1 Conn_ARM_JTAG_SWD_10, Q1 MMBT3904, Q2 AO3401A, Q3 MMBT3904, Q4 AO3401A, SW1 SW_SPDT, SW2 TS-1088-AR02016, U1 STM32F103C8T6, U2 AMS1117-3.3, U3 TJA1040T/CM,118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

Commit message: Add rev0.2 marking to silkscreen
Other:
- board text added: "CANTOTO rev0.2"
Changed lines of the file:
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@@
 		(layer "Edge.Cuts")
+	)
+	(gr_text "CANTOTO rev0.2"
+		(at 40.6 55.2 0)
+		(layer "F.SilkS")
+		(effects
+			(font
+				(size 1.5 1.5)
+				(thickness 0.3)
+				(bold yes)
+			)
+			(justify left bottom)
+		)
 	)
 	(segment
